Commit message: Added sensors to URDFTools.

File: src/test/resources/models/valkyrie/urdf/valkyrie_sim.urdf (robot description, URDF)
Before this commit: robot valkyrie, 78 links, 77 joints
Links:
- link hokuyo_link: mass 0.057664 -> 0.057654
- link leftFoot: mass 2.37 -> 2.27
- link rightFoot: mass 2.37 -> 2.27
- link upperNeckPitchLink: mass 5.30991 -> 3.89
Joints:
- joint leftAnkleRoll: origin xyz=0.0 0.0 0.0 rpy=0.0 0.0 0.0 -> xyz=0.0101259 0.0 0.0 rpy=0.0 0.0 0.0
